File: headphone_dac_proto.sch (KiCad schematic (older format))
At the start: 61 parts

Commit message: Initial component placement finished
Parts:
- removed Y?: 12.288MHz, symbol Device:Crystal
- added Y1: Crystal_GND24, Crystal:Crystal_SMD_Abracon_ABM3B-4Pin_5.0x3.2mm, symbol Device:Crystal_GND24
- C1, C10, C11, C12, C13, C14, C18, C19, C2, C20, C22, C27, C28, C29, C3, C32, C33, C34, C4, C5, C6, C7, C8, C9: renamed from C?; footprint (none) -> Capacitor_SMD:C_0603_1608Metric
- C15, C16, C17, C21, C23, C24, C25, C26, C30, C31: renamed from C?; footprint (none) -> Capacitor_SMD:C_0805_2012Metric
- FB1: renamed from FB?; footprint (none) -> Inductor_SMD:L_0603_1608Metric
- J1: renamed from J?; footprint (none) -> Connector_USB:USB_Mini-B_Wuerth_65100516121_Horizontal
- J2: renamed from J?; footprint (none) -> Connector_PinHeader_2.54mm:PinHeader_2x10_P2.54mm_Vertical
- J3: renamed from J?; footprint (none) -> conn_prog:FTSH-105
- J4, J5: renamed from J?; footprint (none) -> Connector_PinHeader_2.54mm:PinHeader_1x06_P2.54mm_Vertical
- J6: renamed from J?; footprint (none) -> Connector_Audio:Jack_3.5mm_CUI_SJ1-3535NG_Horizontal
- R1, R2, R3, R4, R5, R6, R7, R8, R9: renamed from R?; footprint (none) -> Resistor_SMD:R_0603_1608Metric
- R10: renamed from R?; footprint (none) -> Resistor_THT:R_Axial_DIN0207_L6.3mm_D2.5mm_P15.24mm_Horizontal
- RV1, RV2, RV3: renamed from RV?; footprint (none) -> Connector_PinHeader_2.54mm:PinHeader_1x03_P2.54mm_Vertical
- SW1, SW2: renamed from SW?; footprint (none) -> Button_Switch_Keyboard:SW_Cherry_MX_1.00u_PCB
- gave numbers to parts that had none: 4
Connections:
- wire segments 265 -> 267

Commit message: Change peripheral switches and pots
Parts:
- removed J4: Conn_01x06_Male, Connector_PinHeader_2.54mm:PinHeader_1x06_P2.54mm_Vertical, symbol Connector:Conn_01x06_Male
- added SW3: ~, Button_Switch_THT:SW_PUSH_6mm_H5mm, symbol Switch:SW_Push
- RV1, RV2, RV3: footprint Connector_PinHeader_2.54mm:PinHeader_1x03_P2.54mm_Vertical -> Potentiometer_THT:Potentiometer_Bourns_PTV09A-1_Single_Vertical
- SW1, SW2: footprint Button_Switch_Keyboard:SW_Cherry_MX_1.00u_PCB -> Button_Switch_THT:SW_PUSH_6mm_H5mm
Connections:
- wire segments 267 -> 264
- no-connect marks 38 -> 36
Other:
- note removed: "FTDI 6 pin connector for: TTL-232R-3V3 Cable"
Changed lines of the file:
@@
 F 0 "RV3" H 10100 7950 50  0000 R CNN
 F 1 "100k" V 10100 7900 50  0000 R CNN
-F 2 "Connector_PinHeader_2.54mm:PinHeader_1x03_P2.54mm_Vertical" H 10100 7800 50  0001 C CNN
+F 2 "Potentiometer_THT:Potentiometer_Bourns_PTV09A-1_Single_Vertical" H 10100 7800 50  0001 C CNN
 F 3 "~" H 10100 7800 50  0001 C CNN
 	1    10100 7800
@@
 F 0 "RV2" H 9700 7950 50  0000 R CNN
 F 1 "100k" V 9700 7900 50  0000 R CNN
-F 2 "Connector_PinHeader_2.54mm:PinHeader_1x03_P2.54mm_Vertical" H 9700 7800 50  0001 C CNN
+F 2 "Potentiometer_THT:Potentiometer_Bourns_PTV09A-1_Single_Vertical" H 9700 7800 50  0001 C CNN
 F 3 "~" H 9700 7800 50  0001 C CNN
 	1    9700 7800
@@
 F 0 "RV1" H 9300 7950 50  0000 R CNN
 F 1 "100k" V 9300 7900 50  0000 R CNN
-F 2 "Connector_PinHeader_2.54mm:PinHeader_1x03_P2.54mm_Vertical" H 9300 7800 50  0001 C CNN
+F 2 "Potentiometer_THT:Potentiometer_Bourns_PTV09A-1_Single_Vertical" H 9300 7800 50  0001 C CNN
 F 3 "~" H 9300 7800 50  0001 C CNN
 	1    9300 7800
@@
 Wire Wire Line
 	3250 6100 3550 6100
-$Comp
-L Connector:Conn_01x06_Male J4
-U 1 1 5F3E36AB
-P 5100 4100
-F 0 "J4" H 5072 4074 50  0000 R CNN
-F 1 "Conn_01x06_Male" H 5072 3983 50  0000 R CNN
-F 2 "Connector_PinHeader_2.54mm:PinHeader_1x06_P2.54mm_Vertical" H 5100 4100 50  0001 C CNN
-F 3 "~" H 5100 4100 50  0001 C CNN
-	1    5100 4100
-	-1   0    0    -1
-$EndComp
-$Comp
-L power:GND #PWR0150
-U 1 1 5F3E555D
-P 4700 3900
-F 0 "#PWR0150" H 4700 3650 50  0001 C CNN
-F 1 "GND" V 4700 3650 50  0000 C CNN
-F 2 "" H 4700 3900 50  0001 C CNN
-F 3 "" H 4700 3900 50  0001 C CNN
-	1    4700 3900
-	0    1    -1   0
-$EndComp
-Wire Wire Line
-	4700 3900 4900 3900
-Text Label 4700 4000 0    50   ~ 0
-ft_~cts~
-Text Label 4700 4400 0    50   ~ 0
-ft_~rts~
-Text Label 4700 4300 0    50   ~ 0
-ft_rx
-Text Label 4700 4200 0    50   ~ 0
-ft_tx
-NoConn ~ 4900 4100
-Text Notes 4700 3750 0    50   ~ 0
-FTDI 6 pin connector for: TTL-232R-3V3 Cable
-Wire Wire Line
-	4700 4000 4900 4000
-Wire Wire Line
-	4900 4200 4700 4200
-Wire Wire Line
-	4700 4300 4900 4300
-Wire Wire Line
-	4900 4400 4700 4400
 Text Label 5250 6250 0    50   ~ 0
 bt_rx
@@
 F 0 "SW1" V 4700 6002 50  0000 R CNN
 F 1 "~" V 4655 6002 50  0000 R CNN
-F 2 "Button_Switch_Keyboard:SW_Cherry_MX_1.00u_PCB" H 4700 6250 50  0001 C CNN
+F 2 "Button_Switch_THT:SW_PUSH_6mm_H5mm" H 4700 6250 50  0001 C CNN
 F 3 "~" H 4700 6250 50  0001 C CNN
 	1    4700 6050
@@
 F 0 "SW2" V 4700 6702 50  0000 R CNN
 F 1 "~" V 4655 6702 50  0000 R CNN
-F 2 "Button_Switch_Keyboard:SW_Cherry_MX_1.00u_PCB" H 4700 6950 50  0001 C CNN
+F 2 "Button_Switch_THT:SW_PUSH_6mm_H5mm" H 4700 6950 50  0001 C CNN
 F 3 "~" H 4700 6950 50  0001 C CNN
 	1    4700 6750
@@
 Wire Wire Line
 	6300 5600 6300 5400
-NoConn ~ 6700 5600
 NoConn ~ 6800 5600
 NoConn ~ 8150 7150
@@
 $EndComp
 $Comp
-L power:GND #PWR?
+L power:GND #PWR0163
 U 1 1 5F064196
 P 7200 10000
-F 0 "#PWR?" H 7200 9750 50  0001 C CNN
+F 0 "#PWR0163" H 7200 9750 50  0001 C CNN
 F 1 "GND" V 7200 9750 50  0000 C CNN
 F 2 "" H 7200 10000 50  0001 C CNN
@@
 	7200 10000 7200 9700
 $Comp
-L power:GND #PWR?
+L power:GND #PWR0164
 U 1 1 5F076315
 P 7200 9200
-F 0 "#PWR?" H 7200 8950 50  0001 C CNN
+F 0 "#PWR0164" H 7200 8950 50  0001 C CNN
 F 1 "GND" V 7200 8950 50  0000 C CNN
 F 2 "" H 7200 9200 50  0001 C CNN
@@
 Wire Wire Line
 	7200 9200 7200 9300
+$Comp
+L Switch:SW_Push SW3
+U 1 1 5F00B9F6
+P 6700 4750
+F 0 "SW3" V 6700 4702 50  0000 R CNN
+F 1 "~" V 6655 4702 50  0000 R CNN
+F 2 "Button_Switch_THT:SW_PUSH_6mm_H5mm" H 6700 4950 50  0001 C CNN
+F 3 "~" H 6700 4950 50  0001 C CNN
+	1    6700 4750
+	0    -1   -1   0
+$EndComp
+Wire Wire Line
+	6700 5600 6700 4950
+$Comp
+L power:GND #PWR?
+U 1 1 5F01F914
+P 6700 4450
+F 0 "#PWR?" H 6700 4200 50  0001 C CNN
+F 1 "GND" H 6705 4277 50  0000 C CNN
+F 2 "" H 6700 4450 50  0001 C CNN
+F 3 "" H 6700 4450 50  0001 C CNN
+	1    6700 4450
+	-1   0    0    1
+$EndComp
+Wire Wire Line
+	6700 4450 6700 4550
 $EndSCHEMATC

Commit message: Change all the things
Parts:
- added C35, C36: 1uF, Capacitor_SMD:C_0603_1608Metric, symbol Device:C
Connections:
- net GND: now also C35.2, C36.2
- net at C27.1, RV1.1, RV2.1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: now also C35.1, C36.1
Changed lines of the file:
@@
 	6700 5600 6700 4950
 $Comp
-L power:GND #PWR?
+L power:GND #PWR0150
 U 1 1 5F01F914
 P 6700 4450
-F 0 "#PWR?" H 6700 4200 50  0001 C CNN
+F 0 "#PWR0150" H 6700 4200 50  0001 C CNN
 F 1 "GND" H 6705 4277 50  0000 C CNN
 F 2 "" H 6700 4450 50  0001 C CNN
@@
 Wire Wire Line
 	6700 4450 6700 4550
+$Comp
+L Device:C C35
+U 1 1 5F03BAF0
+P 10500 7800
+F 0 "C35" H 10500 7900 50  0000 L CNN
+F 1 "1uF" H 10500 7700 50  0000 L CNN
+F 2 "Capacitor_SMD:C_0603_1608Metric" H 10538 7650 50  0001 C CNN
+F 3 "~" H 10500 7800 50  0001 C CNN
+	1    10500 7800
+	1    0    0    -1
+$EndComp
+$Comp
+L Device:C C36
+U 1 1 5F03C526
+P 10700 7800
+F 0 "C36" H 10700 7900 50  0000 L CNN
+F 1 "1uF" H 10700 7700 50  0000 L CNN
+F 2 "Capacitor_SMD:C_0603_1608Metric" H 10738 7650 50  0001 C CNN
+F 3 "~" H 10700 7800 50  0001 C CNN
+	1    10700 7800
+	1    0    0    -1
+$EndComp
+Wire Wire Line
+	10300 7550 10500 7550
+Wire Wire Line
+	10500 7550 10500 7650
+Connection ~ 10300 7550
+Wire Wire Line
+	10500 7550 10700 7550
+Wire Wire Line
+	10700 7550 10700 7650
+Connection ~ 10500 7550
+$Comp
+L power:GND #PWR0165
+U 1 1 5F060D79
+P 10500 8050
+F 0 "#PWR0165" H 10500 7800 50  0001 C CNN
+F 1 "GND" V 10500 7800 50  0000 C CNN
+F 2 "" H 10500 8050 50  0001 C CNN
+F 3 "" H 10500 8050 50  0001 C CNN
+	1    10500 8050
+	1    0    0    -1
+$EndComp
+Wire Wire Line
+	10500 8050 10500 7950
+$Comp
+L power:GND #PWR0166
+U 1 1 5F0735D0
+P 10700 8050
+F 0 "#PWR0166" H 10700 7800 50  0001 C CNN
+F 1 "GND" V 10700 7800 50  0000 C CNN
+F 2 "" H 10700 8050 50  0001 C CNN
+F 3 "" H 10700 8050 50  0001 C CNN
+	1    10700 8050
+	1    0    0    -1
+$EndComp
+Wire Wire Line
+	10700 8050 10700 7950
 $EndSCHEMATC

Commit message: Placement is complete. Actually though.
Parts:
- added H1: ~, MountingHole:MountingHole_3mm_Pad_Via, symbol Mechanical:MountingHole_Pad
- added H2, H3, H4: ~, MountingHole:MountingHole_3mm_Pad, symbol Mechanical:MountingHole_Pad
- SW1, SW2, SW3: footprint Button_Switch_THT:SW_PUSH_6mm_H5mm -> Button_Switch_THT:SW_PUSH_6mm_H13mm
Connections:
- net GND: now also H1.1
- no-connect marks 36 -> 39
Changed lines of the file:
@@
 F 0 "SW1" V 4700 6002 50  0000 R CNN
 F 1 "~" V 4655 6002 50  0000 R CNN
-F 2 "Button_Switch_THT:SW_PUSH_6mm_H5mm" H 4700 6250 50  0001 C CNN
+F 2 "Button_Switch_THT:SW_PUSH_6mm_H13mm" H 4700 6250 50  0001 C CNN
 F 3 "~" H 4700 6250 50  0001 C CNN
 	1    4700 6050
@@
 F 0 "SW2" V 4700 6702 50  0000 R CNN
 F 1 "~" V 4655 6702 50  0000 R CNN
-F 2 "Button_Switch_THT:SW_PUSH_6mm_H5mm" H 4700 6950 50  0001 C CNN
+F 2 "Button_Switch_THT:SW_PUSH_6mm_H13mm" H 4700 6950 50  0001 C CNN
 F 3 "~" H 4700 6950 50  0001 C CNN
 	1    4700 6750
@@
 F 0 "SW3" V 6700 4702 50  0000 R CNN
 F 1 "~" V 6655 4702 50  0000 R CNN
-F 2 "Button_Switch_THT:SW_PUSH_6mm_H5mm" H 6700 4950 50  0001 C CNN
+F 2 "Button_Switch_THT:SW_PUSH_6mm_H13mm" H 6700 4950 50  0001 C CNN
 F 3 "~" H 6700 4950 50  0001 C CNN
 	1    6700 4750
@@
 Wire Wire Line
 	10700 8050 10700 7950
+$Comp
+L Mechanical:MountingHole_Pad H1
+U 1 1 5F09ED8B
+P 10500 6550
+F 0 "H1" H 10450 6750 50  0000 L CNN
+F 1 "~" H 10600 6508 50  0000 L CNN
+F 2 "MountingHole:MountingHole_3mm_Pad_Via" H 10500 6550 50  0001 C CNN
+F 3 "~" H 10500 6550 50  0001 C CNN
+	1    10500 6550
+	1    0    0    -1
+$EndComp
+$Comp
+L Mechanical:MountingHole_Pad H2
+U 1 1 5F0A07DF
+P 10700 6550
+F 0 "H2" H 10650 6750 50  0000 L CNN
+F 1 "~" H 10800 6508 50  0000 L CNN
+F 2 "MountingHole:MountingHole_3mm_Pad" H 10700 6550 50  0001 C CNN
+F 3 "~" H 10700 6550 50  0001 C CNN
+	1    10700 6550
+	1    0    0    -1
+$EndComp
+$Comp
+L Mechanical:MountingHole_Pad H3
+U 1 1 5F0A0924
+P 10900 6550
+F 0 "H3" H 10850 6750 50  0000 L CNN
+F 1 "~" H 11000 6508 50  0000 L CNN
+F 2 "MountingHole:MountingHole_3mm_Pad" H 10900 6550 50  0001 C CNN
+F 3 "~" H 10900 6550 50  0001 C CNN
+	1    10900 6550
+	1    0    0    -1
+$EndComp
+$Comp
+L Mechanical:MountingHole_Pad H4
+U 1 1 5F0A0A31
+P 11100 6550
+F 0 "H4" H 11050 6750 50  0000 L CNN
+F 1 "~" H 11200 6508 50  0000 L CNN
+F 2 "MountingHole:MountingHole_3mm_Pad" H 11100 6550 50  0001 C CNN
+F 3 "~" H 11100 6550 50  0001 C CNN
+	1    11100 6550
+	1    0    0    -1
+$EndComp
+NoConn ~ 10700 6650
+NoConn ~ 10900 6650
+NoConn ~ 11100 6650
+$Comp
+L power:GND #PWR0167
+U 1 1 5F0D7C53
+P 10500 6750
+F 0 "#PWR0167" H 10500 6500 50  0001 C CNN
+F 1 "GND" V 10500 6500 50  0000 C CNN
+F 2 "" H 10500 6750 50  0001 C CNN
+F 3 "" H 10500 6750 50  0001 C CNN
+	1    10500 6750
+	1    0    0    -1
+$EndComp
+Wire Wire Line
+	10500 6750 10500 6650
 $EndSCHEMATC

Commit message: I'm sorry Jackson. Please don't read these commit messages
Parts:
- removed J5: Conn_01x06, Connector_PinHeader_2.54mm:PinHeader_1x06_P2.54mm_Vertical, symbol Connector_Generic:Conn_01x06
Connections:
- net i2s_sd is gone; now on net i2s_sdo: U3.1 (SDIN)
- net bt_cts: no longer U2.66 (P2[4])
- net bt_rts: no longer U2.1 (P2[6])
- net bt_rx: no longer U2.2 (P2[7])
- net bt_tx: no longer U2.68 (P2[5])
- net i2s_lrck: now also U2.68 (P2[5]); no longer U2.49 (P0[1])
- net i2s_mck: now also U2.66 (P2[4]); no longer U2.48 (P0[0])
- net i2s_sck: now also U2.1 (P2[6]); no longer U2.50 (P0[2])
- net i2s_sdo: now also U2.2 (P2[7]); no longer U2.51 (P0[3])
- net sw1: now reaches SW1.1
- net sw1: now also U2.4 (P12[5]); no longer U2.3 (P12[4])
- net sw2: now reaches SW2.2
- net sw2: now also U2.3 (P12[4]); no longer U2.4 (P12[5])
- net at U2.61 (P15[5]): no longer SW3.1
- net i2s_sdi: no longer names the net of U2.53 (P0[4])
- new net sw3: SW3.1
Other:
- note removed: "I2S Bus Connector"
- moved on the sheet: SW1, SW2, SW3
Changed lines of the file:
@@
 $EndComp
 Text Label 8400 1900 0    50   ~ 0
-i2s_sd
+i2s_sdo
 Text Label 8400 2000 0    50   ~ 0
 i2s_sck
@@
 Text Notes 7600 9750 0    50   ~ 0
 Stray Capacitance: 2pF\nLoad Capacitance (Crystal): 10pF\nShunt Capacitance (Crystal): 7pF
-Text Label 8450 6450 2    50   ~ 0
+Text Label 6200 5300 3    50   ~ 0
 i2s_mck
-Text Label 8450 6350 2    50   ~ 0
+Text Label 6000 5300 3    50   ~ 0
 i2s_lrck
-Text Label 8450 6250 2    50   ~ 0
+Text Label 5150 6150 0    50   ~ 0
 i2s_sck
-Text Label 8450 6150 2    50   ~ 0
+Text Label 5150 6250 0    50   ~ 0
 i2s_sdo
 Wire Wire Line
@@
 Wire Wire Line
 	8150 6450 8450 6450
-Text Label 7500 5300 3    50   ~ 0
-i2s_sdi
 Wire Wire Line
 	7500 5300 7500 5600
@@
 Wire Wire Line
 	3250 6100 3550 6100
-Text Label 5250 6250 0    50   ~ 0
+Text Label 5250 5500 0    50   ~ 0
 bt_rx
 Wire Wire Line
-	5250 6250 5450 6250
-Text Label 5250 6150 0    50   ~ 0
+	5150 6250 5450 6250
+Text Label 5250 5400 0    50   ~ 0
 bt_rts
 Wire Wire Line
-	5250 6150 5450 6150
-Text Label 6000 5400 3    50   ~ 0
+	5150 6150 5450 6150
+Text Label 5000 5050 3    50   ~ 0
 bt_tx
-Text Label 6200 5400 3    50   ~ 0
+Text Label 5250 5600 0    50   ~ 0
 bt_cts
 Wire Wire Line
-	6200 5400 6200 5600
-Wire Wire Line
-	6000 5600 6000 5400
+	6200 5300 6200 5600
+Wire Wire Line
+	6000 5600 6000 5300
 $Comp
 L Switch:SW_Push SW1
 U 1 1 5F4EBD7A
-P 4700 6050
-F 0 "SW1" V 4700 6002 50  0000 R CNN
-F 1 "~" V 4655 6002 50  0000 R CNN
-F 2 "Button_Switch_THT:SW_PUSH_6mm_H13mm" H 4700 6250 50  0001 C CNN
-F 3 "~" H 4700 6250 50  0001 C CNN
-	1    4700 6050
-	0    -1   -1   0
+P 3800 5200
+F 0 "SW1" V 3800 5152 50  0000 R CNN
+F 1 "~" V 3755 5152 50  0000 R CNN
+F 2 "Button_Switch_THT:SW_PUSH_6mm_H13mm" H 3800 5400 50  0001 C CNN
+F 3 "~" H 3800 5400 50  0001 C CNN
+	1    3800 5200
+	0    1    -1   0
 $EndComp
 $Comp
 L Switch:SW_Push SW2
 U 1 1 5F4ED23B
-P 4700 6750
-F 0 "SW2" V 4700 6702 50  0000 R CNN
-F 1 "~" V 4655 6702 50  0000 R CNN
-F 2 "Button_Switch_THT:SW_PUSH_6mm_H13mm" H 4700 6950 50  0001 C CNN
-F 3 "~" H 4700 6950 50  0001 C CNN
-	1    4700 6750
-	0    -1   -1   0
-$EndComp
-Wire Wire Line
-	4700 6550 4700 6450
-Wire Wire Line
-	4700 6450 5450 6450
-Wire Wire Line
-	5450 6350 4700 6350
-Wire Wire Line
-	4700 6350 4700 6250
+P 4250 5200
+F 0 "SW2" V 4250 5152 50  0000 R CNN
+F 1 "~" V 4205 5152 50  0000 R CNN
+F 2 "Button_Switch_THT:SW_PUSH_6mm_H13mm" H 4250 5400 50  0001 C CNN
+F 3 "~" H 4250 5400 50  0001 C CNN
+	1    4250 5200
+	0    1    1    0
+$EndComp
+Wire Wire Line
+	4250 5400 4250 5500
+Wire Wire Line
+	5450 6350 5150 6350
+Wire Wire Line
+	3800 5500 3800 5400
 $Comp
 L power:GND #PWR0151
 U 1 1 5F50471B
-P 4700 7050
-F 0 "#PWR0151" H 4700 6800 50  0001 C CNN
-F 1 "GND" H 4705 6877 50  0000 C CNN
-F 2 "" H 4700 7050 50  0001 C CNN
-F 3 "" H 4700 7050 50  0001 C CNN
-	1    4700 7050
-	1    0    0    -1
-$EndComp
-Wire Wire Line
-	4700 7050 4700 6950
+P 4250 4900
+F 0 "#PWR0151" H 4250 4650 50  0001 C CNN
+F 1 "GND" H 4255 4727 50  0000 C CNN
+F 2 "" H 4250 4900 50  0001 C CNN
+F 3 "" H 4250 4900 50  0001 C CNN
+	1    4250 4900
+	-1   0    0    1
+$EndComp
+Wire Wire Line
+	4250 4900 4250 5000
 $Comp
 L power:GND #PWR0152
 U 1 1 5F510616
-P 4700 5750
-F 0 "#PWR0152" H 4700 5500 50  0001 C CNN
-F 1 "GND" H 4705 5577 50  0000 C CNN
-F 2 "" H 4700 5750 50  0001 C CNN
-F 3 "" H 4700 5750 50  0001 C CNN
-	1    4700 5750
-	-1   0    0    1
-$EndComp
-Wire Wire Line
-	4700 5750 4700 5850
+P 3800 4900
+F 0 "#PWR0152" H 3800 4650 50  0001 C CNN
+F 1 "GND" H 3805 4727 50  0000 C CNN
+F 2 "" H 3800 4900 50  0001 C CNN
+F 3 "" H 3800 4900 50  0001 C CNN
+	1    3800 4900
+	1    0    0    1
+$EndComp
+Wire Wire Line
+	3800 4900 3800 5000
 Text Label 5200 7050 0    50   ~ 0
 xres
@@
 Analog Inputs
 $Comp
-L Connector_Generic:Conn_01x06 J5
-U 1 1 5F8492FD
-P 9050 3950
-F 0 "J5" H 9130 3942 50  0000 L CNN
-F 1 "Conn_01x06" H 9130 3851 50  0000 L CNN
-F 2 "Connector_PinHeader_2.54mm:PinHeader_1x06_P2.54mm_Vertical" H 9050 3950 50  0001 C CNN
-F 3 "~" H 9050 3950 50  0001 C CNN
-	1    9050 3950
-	1    0    0    -1
-$EndComp
-$Comp
-L power:GND #PWR0155
-U 1 1 5F84A676
-P 8650 3750
-F 0 "#PWR0155" H 8650 3500 50  0001 C CNN
-F 1 "GND" V 8650 3500 50  0000 C CNN
-F 2 "" H 8650 3750 50  0001 C CNN
-F 3 "" H 8650 3750 50  0001 C CNN
-	1    8650 3750
-	0    1    1    0
-$EndComp
-Wire Wire Line
-	8650 3750 8850 3750
-$Comp
-L power:+3.3V #PWR0156
-U 1 1 5F85A280
-P 8650 3850
-F 0 "#PWR0156" H 8650 3700 50  0001 C CNN
-F 1 "+3.3V" V 8650 4100 50  0000 C CNN
-F 2 "" H 8650 3850 50  0001 C CNN
-F 3 "" H 8650 3850 50  0001 C CNN
-	1    8650 3850
-	0    -1   -1   0
-$EndComp
-Wire Wire Line
-	8650 3850 8850 3850
-Text Label 8550 3950 0    50   ~ 0
-i2s_sd
-Text Label 8550 4050 0    50   ~ 0
-i2s_sck
-Text Label 8550 4150 0    50   ~ 0
-i2s_lrck
-Wire Wire Line
-	8850 4150 8550 4150
-Wire Wire Line
-	8550 4050 8850 4050
-Wire Wire Line
-	8850 3950 8550 3950
-Text Label 8550 4250 0    50   ~ 0
-i2s_mck
-Wire Wire Line
-	8550 4250 8850 4250
-$Comp
 L audio_amplifier:TPA6139A2 U4
 U 1 1 5F8BD36E
@@
 Text Notes 13650 750  0    50   ~ 0
 Headphone Connector
-Wire Notes Line
-	8150 3450 9950 3450
-Wire Notes Line
-	9950 3450 9950 4500
-Wire Notes Line
-	9950 4500 8150 4500
-Wire Notes Line
-	8150 4500 8150 3450
-Text Notes 8150 3450 0    50   ~ 0
-I2S Bus Connector
 $Comp
 L Connector:AudioJack3 J6
@@
 L Switch:SW_Push SW3
 U 1 1 5F00B9F6
-P 6700 4750
-F 0 "SW3" V 6700 4702 50  0000 R CNN
-F 1 "~" V 6655 4702 50  0000 R CNN
-F 2 "Button_Switch_THT:SW_PUSH_6mm_H13mm" H 6700 4950 50  0001 C CNN
-F 3 "~" H 6700 4950 50  0001 C CNN
-	1    6700 4750
-	0    -1   -1   0
-$EndComp
-Wire Wire Line
-	6700 5600 6700 4950
+P 4600 5200
+F 0 "SW3" V 4600 5152 50  0000 R CNN
+F 1 "~" V 4555 5152 50  0000 R CNN
+F 2 "Button_Switch_THT:SW_PUSH_6mm_H13mm" H 4600 5400 50  0001 C CNN
+F 3 "~" H 4600 5400 50  0001 C CNN
+	1    4600 5200
+	0    1    -1   0
+$EndComp
+Wire Wire Line
+	4600 5500 4600 5400
 $Comp
 L power:GND #PWR0150
 U 1 1 5F01F914
-P 6700 4450
-F 0 "#PWR0150" H 6700 4200 50  0001 C CNN
-F 1 "GND" H 6705 4277 50  0000 C CNN
-F 2 "" H 6700 4450 50  0001 C CNN
-F 3 "" H 6700 4450 50  0001 C CNN
-	1    6700 4450
-	-1   0    0    1
-$EndComp
-Wire Wire Line
-	6700 4450 6700 4550
+P 4600 4900
+F 0 "#PWR0150" H 4600 4650 50  0001 C CNN
+F 1 "GND" H 4605 4727 50  0000 C CNN
+F 2 "" H 4600 4900 50  0001 C CNN
+F 3 "" H 4600 4900 50  0001 C CNN
+	1    4600 4900
+	1    0    0    1
+$EndComp
+Wire Wire Line
+	4600 4900 4600 5000
 $Comp
 L Device:C C35
@@
 Wire Wire Line
 	10500 6750 10500 6650
+Text Label 3800 5500 1    50   ~ 0
+sw1
+Text Label 4250 5500 1    50   ~ 0
+sw2
+Text Label 4600 5500 1    50   ~ 0
+sw3
+Text Label 5150 6450 0    50   ~ 0
+sw1
+Wire Wire Line
+	5150 6450 5450 6450
+Text Label 5150 6350 0    50   ~ 0
+sw2
 $EndSCHEMATC

Commit message: Started routing
Connections:
- net ft_rx is gone; now on net sw3: U2.63 (P2[1])
- net ft_tx is gone; now on net sw2: U2.64 (P2[2])
- net ft_~cts~ is gone; now on net sw1: U2.65 (P2[3])
- net ft_~rts~ is gone; now on net bt_rts: U2.62 (P2[0])
- net a0: now also U2.34 (P3[5]); no longer U2.36 (P3[6])
- net a1: now also U2.36 (P3[6]); no longer U2.34 (P3[5])
- net a2: now also U2.37 (P3[7]); no longer U2.33 (P3[4])
- net bt_cts: now also U2.61 (P15[5])
- net bt_rx: now also U2.4 (P12[5])
- net bt_tx: now also U2.3 (P12[4])
- net sw1: no longer U2.4 (P12[5])
- net sw2: no longer U2.3 (P12[4])
- net as: now reaches C27.1, C35.1, C36.1, RV1.1, RV2.1, RV3.1
- net as: now also U2.33 (P3[4]); no longer U2.37 (P3[7])
- no-connect marks 39 -> 44
Changed lines of the file:
@@
 Connection ~ 3900 1650
 Wire Wire Line
-	3900 1650 4800 1650
+	3900 1650 4000 1650
 $Comp
 L power:GND #PWR0107
@@
 Text Label 5150 6250 0    50   ~ 0
 i2s_sdo
-Wire Wire Line
-	8450 6150 8150 6150
-Wire Wire Line
-	8150 6250 8450 6250
-Wire Wire Line
-	8450 6350 8150 6350
-Wire Wire Line
-	8150 6450 8450 6450
-Wire Wire Line
-	7500 5300 7500 5600
 $Comp
 L Device:R_POT RV3
@@
 $EndComp
 Wire Wire Line
-	8150 7550 9300 7550
-Wire Wire Line
 	10100 7550 10100 7650
 $Comp
@@
 Wire Wire Line
 	9300 7650 9300 7550
-Connection ~ 9300 7550
 Wire Wire Line
 	9300 7550 9700 7550
@@
 Wire Wire Line
 	9050 7800 9150 7800
+Text Label 7600 8500 1    50   ~ 0
+a0
+Wire Wire Line
+	8350 7650 8150 7650
 Text Label 8350 7650 2    50   ~ 0
-a0
-Wire Wire Line
-	8350 7650 8150 7650
-Text Label 7600 8500 1    50   ~ 0
 a1
 Wire Wire Line
 	7600 8500 7600 8300
-Text Label 7500 8500 1    50   ~ 0
+Text Label 8350 7550 2    50   ~ 0
 a2
 Wire Wire Line
@@
 Wire Wire Line
 	3250 6100 3550 6100
-Text Label 5250 5500 0    50   ~ 0
+Text Label 5150 6450 0    50   ~ 0
 bt_rx
 Wire Wire Line
 	5150 6250 5450 6250
-Text Label 5250 5400 0    50   ~ 0
+Text Label 6600 5400 3    50   ~ 0
 bt_rts
 Wire Wire Line
 	5150 6150 5450 6150
-Text Label 5000 5050 3    50   ~ 0
+Text Label 5150 6350 0    50   ~ 0
 bt_tx
-Text Label 5250 5600 0    50   ~ 0
+Text Label 6700 5400 3    50   ~ 0
 bt_cts
 Wire Wire Line
@@
 Wire Wire Line
 	3200 8900 3200 8800
-Text Label 6300 5400 3    50   ~ 0
-ft_~cts~
-Text Label 6400 5400 3    50   ~ 0
-ft_tx
-Text Label 6500 5400 3    50   ~ 0
-ft_rx
-Text Label 6600 5400 3    50   ~ 0
-ft_~rts~
 Wire Wire Line
 	6600 5400 6600 5600
@@
 Text Label 4600 5500 1    50   ~ 0
 sw3
-Text Label 5150 6450 0    50   ~ 0
+Text Label 6300 5400 3    50   ~ 0
 sw1
 Wire Wire Line
 	5150 6450 5450 6450
-Text Label 5150 6350 0    50   ~ 0
+Text Label 6400 5400 3    50   ~ 0
 sw2
+NoConn ~ 7500 5600
+NoConn ~ 8150 6450
+NoConn ~ 8150 6350
+NoConn ~ 8150 6250
+NoConn ~ 8150 6150
+Text Label 6500 5400 3    50   ~ 0
+sw3
+Wire Wire Line
+	6700 5400 6700 5600
+$Comp
+L power:PWR_FLAG #FLG0101
+U 1 1 5F3757E1
+P 4000 1550
+F 0 "#FLG0101" H 4000 1625 50  0001 C CNN
+F 1 "PWR_FLAG" H 4000 1723 50  0001 C CNN
+F 2 "" H 4000 1550 50  0001 C CNN
+F 3 "~" H 4000 1550 50  0001 C CNN
+	1    4000 1550
+	1    0    0    -1
+$EndComp
+Wire Wire Line
+	4000 1550 4000 1650
+Connection ~ 4000 1650
+Wire Wire Line
+	4000 1650 4800 1650
+Text Label 7500 8500 1    50   ~ 0
+as
+Wire Wire Line
+	8150 7550 8350 7550
+Text Label 10700 7550 2    50   ~ 0
+as
 $EndSCHEMATC
