File: headphone_dac_proto.sch (KiCad schematic (older format))
At the start: 66 parts, among them J1 USB_B_Mini, J2 Conn_02x10_Odd_Even, J3 Conn_02x05_Odd_Even, J6 6.35mm, U1 LT3042xMSE, U2 CY8C5888LTI-LP097, U3 CS4344, U4 TPA6139A2, Y1 Crystal_GND24

Commit message: ERC and DRC passing
Parts:
- U1: footprint Package_SO:MSOP-10-1EP_3x3mm_P0.5mm_EP1.68x1.88mm -> Package_SO:MSOP-10-1EP_3x3mm_P0.5mm_EP1.68x1.88mm_ThermalVias
Changed lines of the file:
@@
 F 0 "U1" H 5300 2117 50  0000 C CNN
 F 1 "LT3042xMSE" H 5300 2026 50  0000 C CNN
-F 2 "Package_SO:MSOP-10-1EP_3x3mm_P0.5mm_EP1.68x1.88mm" H 5300 2075 50  0001 C CNN
+F 2 "Package_SO:MSOP-10-1EP_3x3mm_P0.5mm_EP1.68x1.88mm_ThermalVias" H 5300 2075 50  0001 C CNN
 F 3 "https://www.analog.com/media/en/technical-documentation/data-sheets/3042fb.pdf" H 5300 1750 50  0001 C CNN
 	1    5300 1750
@@
 Wire Wire Line
 	9050 7800 9150 7800
-Text Label 7600 8500 1    50   ~ 0
-a0
 Wire Wire Line
 	8350 7650 8150 7650
@@
 Headphone Connector
 $Comp
-L Connector:AudioJack3 J6
-U 1 1 5F017100
-P 14300 2000
-F 0 "J6" H 14020 2025 50  0000 R CNN
-F 1 "6.35mm" H 14020 1934 50  0000 R CNN
-F 2 "Connector_Audio:Jack_3.5mm_CUI_SJ1-3535NG_Horizontal" H 14300 2000 50  0001 C CNN
-F 3 "~" H 14300 2000 50  0001 C CNN
-	1    14300 2000
-	-1   0    0    1
-$EndComp
-$Comp
 L Device:Crystal_GND24 Y1
 U 1 1 5F038FE4
@@
 Wire Wire Line
 	4000 1650 4800 1650
-Text Label 7500 8500 1    50   ~ 0
-as
 Wire Wire Line
 	8150 7550 8350 7550
 Text Label 10700 7550 2    50   ~ 0
 as
+Text Label 7600 8500 1    50   ~ 0
+a0
+Text Label 7500 8500 1    50   ~ 0
+as
+$Comp
+L Connector:AudioJack3 J6
+U 1 1 5F017100
+P 14300 2000
+F 0 "J6" H 14020 2025 50  0000 R CNN
+F 1 "6.35mm" H 14020 1934 50  0000 R CNN
+F 2 "Connector_Audio:Jack_3.5mm_CUI_SJ1-3535NG_Horizontal" H 14300 2000 50  0001 C CNN
+F 3 "~" H 14300 2000 50  0001 C CNN
+	1    14300 2000
+	-1   0    0    1
+$EndComp
 $EndSCHEMATC

Commit message: More cleanup
Parts:
- J2: value Conn_02x10_Odd_Even -> Bluetooth
- J3: value Conn_02x05_Odd_Even -> Prog
- J6: value 6.35mm -> Headphones
Connections:
- net bt_cts: no longer U2.61 (P15[5])
- net bt_rts: no longer U2.62 (P2[0])
- no-connect marks 44 -> 48
Changed lines of the file:
@@
 P 2950 6400
 F 0 "J2" H 3000 5675 50  0000 C CNN
-F 1 "Conn_02x10_Odd_Even" H 3000 5766 50  0000 C CNN
+F 1 "Bluetooth" H 3000 5766 50  0000 C CNN
 F 2 "Connector_PinHeader_2.54mm:PinHeader_2x10_P2.54mm_Vertical" H 2950 6400 50  0001 C CNN
 F 3 "~" H 2950 6400 50  0001 C CNN
@@
 Wire Wire Line
 	5150 6250 5450 6250
-Text Label 6600 5400 3    50   ~ 0
-bt_rts
 Wire Wire Line
 	5150 6150 5450 6150
 Text Label 5150 6350 0    50   ~ 0
 bt_tx
-Text Label 6700 5400 3    50   ~ 0
-bt_cts
 Wire Wire Line
 	6200 5300 6200 5600
@@
 P 3500 8700
 F 0 "J3" H 3550 9117 50  0000 C CNN
-F 1 "Conn_02x05_Odd_Even" H 3550 9026 50  0000 C CNN
+F 1 "Prog" H 3550 9026 50  0000 C CNN
 F 2 "conn_prog:FTSH-105" H 3500 8700 50  0001 C CNN
 F 3 "~" H 3500 8700 50  0001 C CNN
@@
 Wire Wire Line
 	3200 8900 3200 8800
-Wire Wire Line
-	6600 5400 6600 5600
 Wire Wire Line
 	6500 5600 6500 5400
@@
 Text Label 6500 5400 3    50   ~ 0
 sw3
-Wire Wire Line
-	6700 5400 6700 5600
 $Comp
 L power:PWR_FLAG #FLG0101
@@
 P 14300 2000
 F 0 "J6" H 14020 2025 50  0000 R CNN
-F 1 "6.35mm" H 14020 1934 50  0000 R CNN
+F 1 "Headphones" H 14020 1934 50  0000 R CNN
 F 2 "Connector_Audio:Jack_3.5mm_CUI_SJ1-3535NG_Horizontal" H 14300 2000 50  0001 C CNN
 F 3 "~" H 14300 2000 50  0001 C CNN
@@
 	-1   0    0    1
 $EndComp
+NoConn ~ 2450 6200
+NoConn ~ 6600 5600
+NoConn ~ 6700 5600
+NoConn ~ 2450 6300
 $EndSCHEMATC
